Commit message: Added inertia and collisions

File: src/rc_car_description/urdf/robot_core.xacro (robot description, xacro)
@@ -1,4 +1,5 @@
 <?xml version="1.0"?>
 <robot xmlns:xacro="http://www.ros.org/wiki/xacro" >
+    <xacro:include filename="inertial_macros.xacro" />
     <material name="blue">
         <color rgba="0 0 1 1" />
@@ -19,4 +20,13 @@
             <material name="green" />
         </visual>
+        <collision>
+            <geometry>
+                <box size="0.6 0.4 0.2" />
+            </geometry>
+            <origin xyz="0 0 0.1" rpy="0 0 0" />
+        </collision>
+        <xacro:inertial_box mass="0.5" x="0.6" y="0.4" z="0.2">
+            <origin xyz="0 0 0.1" rpy="0 0 0" />
+        </xacro:inertial_box>
     </link>
     <joint name="base_joint" type="fixed">
@@ -33,4 +43,13 @@
             <material name="blue" />
         </visual>
+        <collision>
+            <geometry>
+                <cylinder radius="0.1" length="0.05" />
+            </geometry>
+            <origin xyz="0 0 0" rpy="0 0 0" />
+        </collision>
+        <xacro:inertial_cylinder mass="0.1" radius="0.1" length="0.05" >
+            <origin xyz="0 0 0" rpy="0 0 0" />
+        </xacro:inertial_cylinder>
     </link>
     <joint name="base_lidar_joint" type="fixed">
@@ -47,4 +66,13 @@
             <material name="grey" />
         </visual>
+        <collision>
+            <geometry>
+                <cylinder radius="0.1" length="0.05" />
+            </geometry>
+            <origin xyz="0 0 0" rpy="1.57 0 0" />
+        </collision>
+        <xacro:inertial_cylinder mass="0.1" radius="0.1" length="0.05" >
+            <origin xyz="0 0 0" rpy="1.57 0 0" />
+        </xacro:inertial_cylinder>
     </link>
     <joint name="base_left_wheel_joint" type="continuous">
@@ -62,4 +90,13 @@
             <material name="grey" />
         </visual>
+        <collision>
+            <geometry>
+                <cylinder radius="0.1" length="0.05" />
+            </geometry>
+            <origin xyz="0 0 0" rpy="1.57 0 0" />
+        </collision>
+        <xacro:inertial_cylinder mass="0.1" radius="0.1" length="0.05" >
+            <origin xyz="0 0 0" rpy="1.57 0 0" />
+        </xacro:inertial_cylinder>
     </link>
     <joint name="base_right_wheel_joint" type="continuous">
@@ -77,4 +114,13 @@
             <material name="grey" />
         </visual>
+        <collision>
+            <geometry>
+                <sphere radius="0.05" />
+            </geometry>
+            <origin xyz="0 0 0" rpy="0 0 0" />
+        </collision>
+        <xacro:inertial_sphere mass="0.1" radius="0.05">
+            <origin xyz="0 0 0" rpy="0 0 0" />
+        </xacro:inertial_sphere>
     </link>
     <joint name="joint_name" type="fixed">
